Commit message: add joint limit and let IK solver satisfy

File: rby1_description/urdf/rby1.urdf (robot description, URDF)
Before this commit: robot rby1, 37 links, 36 joints
Joints:
- joint left_arm_0: limit lower=-3.141592654 upper=3.141592654 effort=70.0 velocity=3.141592654 -> lower=-2.356194490 upper=2.356194490 effort=70.0 velocity=3.141592654
- joint left_arm_1: limit lower=-0.017453293 upper=3.141592654 effort=70.0 velocity=3.141592654 -> lower=0.0 upper=3.141592654 effort=70.0 velocity=3.141592654
- joint left_arm_2: limit lower=-3.141592654 upper=3.141592654 effort=70.0 velocity=3.141592654 -> lower=-2.094395102 upper=2.094395102 effort=70.0 velocity=3.141592654
- joint left_arm_3: limit lower=-2.617993878 upper=0.017453293 effort=40.0 velocity=3.141592654 -> lower=-2.617993878 upper=0.0 effort=40.0 velocity=3.141592654
- joint left_arm_4: limit lower=-3.141592654 upper=3.141592654 effort=10.0 velocity=6.283185308 -> lower=-6.283185307 upper=6.283185307 effort=10.0 velocity=6.283185308
- joint left_arm_5: limit lower=-1.570796327 upper=1.919862177 effort=10.0 velocity=6.283185308 -> lower=-1.745329252 upper=2.007128640 effort=10.0 velocity=6.283185308
- joint left_arm_6: limit lower=-2.792526803 upper=2.792526803 effort=8.0 velocity=2.094395102 -> lower=-2.967059728 upper=2.967059728 effort=8.0 velocity=6.283185308
- joint right_arm_0: limit lower=-3.141592654 upper=3.141592654 effort=70.0 velocity=3.141592654 -> lower=-2.356194490 upper=2.356194490 effort=70.0 velocity=3.141592654
- joint right_arm_1: limit lower=-3.141592654 upper=0.017453293 effort=70.0 velocity=3.141592654 -> lower=-3.141592654 upper=0.0 effort=70.0 velocity=3.141592654
- joint right_arm_2: limit lower=-3.141592654 upper=3.141592654 effort=70.0 velocity=3.141592654 -> lower=-2.094395102 upper=2.094395102 effort=70.0 velocity=3.141592654
- joint right_arm_3: limit lower=-2.617993878 upper=0.017453293 effort=40.0 velocity=3.141592654 -> lower=-2.617993878 upper=0.0 effort=40.0 velocity=3.141592654
- joint right_arm_4: limit lower=-3.141592654 upper=3.141592654 effort=10.0 velocity=6.283185308 -> lower=-6.283185307 upper=6.283185307 effort=10.0 velocity=6.283185308
- joint right_arm_5: limit lower=-1.570796327 upper=1.919862177 effort=10.0 velocity=6.283185308 -> lower=-1.745329252 upper=2.007128640 effort=10.0 velocity=6.283185308
- joint right_arm_6: limit lower=-2.792526803 upper=2.792526803 effort=8.0 velocity=2.094395102 -> lower=-2.967059728 upper=2.967059728 effort=8.0 velocity=6.283185308
- joint torso_0: limit lower=-0.261799388 upper=0.261799388 effort=270.0 velocity=2.09439510 -> lower=-0.349065850 upper=0.349065850 effort=270.0 velocity=2.09439510
- joint torso_1: limit lower=-0.523598776 upper=1.570796327 effort=270.0 velocity=2.09439510 -> lower=-1.047197551 upper=1.221730476 effort=270.0 velocity=2.09439510
- joint torso_2: limit lower=-2.617993878 upper=1.570796327 effort=270.0 velocity=2.09439510 -> lower=-2.443460953 upper=0.785398163 effort=270.0 velocity=3.141592654
- joint torso_5: limit lower=-2.35619449 upper=2.35619449 effort=120.0 velocity=3.141592654 -> lower=-1.570796327 upper=1.570796327 effort=120.0 velocity=3.141592654

Commit message: add parallel gripper joint

File: rby1_description/urdf/rby1.urdf (robot description, URDF)
Before this commit: robot rby1, 37 links, 36 joints
Joints:
- joint gripper_finger_l1: type fixed -> prismatic
- joint gripper_finger_l2: mimic (none) -> joint=gripper_finger_l1 multiplier=-1 offset=0; type fixed -> prismatic
- joint gripper_finger_r1: type fixed -> prismatic
- joint gripper_finger_r2: mimic (none) -> joint=gripper_finger_r1 multiplier=-1 offset=0; type fixed -> prismatic
