Commit message: add rby1a_1_2 usd

File: rby1_description/urdf/rby1a/model_v1_2.urdf (robot description, URDF)
Before this commit: robot RBY1_A_v1_2, 34 links, 33 joints
Joints:
- joint gripper_finger_l2_joint: mimic joint=gripper_finger_l1_joint multiplier=1.0 offset=0.0 -> joint=gripper_finger_l1_joint multiplier=-1.0 offset=0.0
- joint gripper_finger_r2_joint: mimic joint=gripper_finger_r1_joint multiplier=1.0 offset=0.0 -> joint=gripper_finger_r1_joint multiplier=-1.0 offset=0.0

Commit message: update rby1 usd

File: rby1_description/urdf/rby1a/model_v1_2.urdf (robot description, URDF)
Before this commit: robot RBY1_A_v1_2, 34 links, 33 joints
Links:
- link gripper_left: geometry collision mesh filename=package://rby1_description/meshes/rby1a/parallel_gripper_wr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 scale=0.001 0.001 0.001; visual mesh filename=package://rby1_description/meshes/rby1a/parallel_gripper_wr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 scale=0.001 0.001 0.001
- link gripper_right: geometry collision mesh filename=package://rby1_description/meshes/rby1a/parallel_gripper_wr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 scale=0.001 0.001 0.001; visual mesh filename=package://rby1_description/meshes/rby1a/parallel_gripper_wr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 scale=0.001 0.001 0.001
Joints:
- joint gripper_finger_l1_joint: origin xyz=0.003 0.0 -0.075 rpy=0.0 0.0 0.0 -> xyz=0.003 0.0 -0.022 rpy=0.0 0.0 0.0
- joint gripper_finger_l2_joint: origin xyz=-0.003 0.0 -0.075 rpy=0.0 0.0 3.1415926535 -> xyz=-0.003 0.0 -0.022 rpy=0.0 0.0 3.1415926535
- joint gripper_finger_r1_joint: origin xyz=0.003 0.0 -0.075 rpy=0.0 0.0 0.0 -> xyz=0.003 0.0 -0.022 rpy=0.0 0.0 0.0
- joint gripper_finger_r2_joint: origin xyz=-0.003 0.0 -0.075 rpy=0.0 0.0 3.1415926535 -> xyz=-0.003 0.0 -0.022 rpy=0.0 0.0 3.1415926535
- joint gripper_left_joint: origin xyz=0.0 0.0 0.012 rpy=0 0.0 0.0 -> xyz=0.0 0.0 -0.04 rpy=0 0.0 3.1415926535
- joint gripper_right_joint: origin xyz=0.0 0.0 0.012 rpy=0 0.0 0.0 -> xyz=0.0 0.0 -0.04 rpy=0 0.0 0.0

Commit message: detach d405 cam

File: rby1_description/urdf/rby1a/model_v1_2.urdf (robot description, URDF)
Before this commit: robot RBY1_A_v1_2, 34 links, 33 joints
Links:
- added link d405_link_l; collision mesh filename=package://rby1_description/meshes/rby1a/D405.dae; visual mesh filename=package://rby1_description/meshes/rby1a/D405.dae
- added link d405_link_r; collision mesh filename=package://rby1_description/meshes/rby1a/D405.dae; visual mesh filename=package://rby1_description/meshes/rby1a/D405.dae
- link gripper_left: geometry collision mesh filename=package://rby1_description/meshes/rby1a/GRIPPER_BODY.dae; visual mesh filename=package://rby1_description/meshes/rby1a/GRIPPER_BODY.dae
- link gripper_right: geometry collision mesh filename=package://rby1_description/meshes/rby1a/GRIPPER_BODY.dae; visual mesh filename=package://rby1_description/meshes/rby1a/GRIPPER_BODY.dae
Joints:
- added joint d405_joint_l: type fixed, parent gripper_left, child d405_link_l, origin xyz=0 0 0 rpy=0 0 0
- added joint d405_joint_r: type fixed, parent gripper_right, child d405_link_r, origin xyz=0 0 0 rpy=0 0 0
